File: pcb/pcb.kicad_pcb (KiCad board)
At the start: 2 copper layers, 332.3 x 332.3 mm, 2 parts, among them U1 MOUDLE-SEEEDUINO-XIAO-ESP32S3

Commit message: Moving along
Parts:
- added BT1: Battery Connector, Connector_JST:JST_PH_S2B-PH-K_1x02_P2.00mm_Horizontal, B.Cu at (315.1, 320.4)
- added D1: WS2812C-2020, LED_SMD:LED_WS2812B-2020_PLCC4_2.0x2.0mm, F.Cu at (370.6, 176.4)
- added D10: WS2812C-2020, LED_SMD:LED_WS2812B-2020_PLCC4_2.0x2.0mm, F.Cu at (228.2, 175.3)
- added D11: WS2812C-2020, LED_SMD:LED_WS2812B-2020_PLCC4_2.0x2.0mm, F.Cu at (312.0, 180.5)
- added D12: WS2812C-2020, LED_SMD:LED_WS2812B-2020_PLCC4_2.0x2.0mm, F.Cu at (324.7, 189.7)
- added D13: WS2812C-2020, LED_SMD:LED_WS2812B-2020_PLCC4_2.0x2.0mm, F.Cu at (237.0, 245.3)
- added D14: WS2812C-2020, LED_SMD:LED_WS2812B-2020_PLCC4_2.0x2.0mm, F.Cu at (350.0, 185.0)
- added D15: WS2812C-2020, LED_SMD:LED_WS2812B-2020_PLCC4_2.0x2.0mm, F.Cu at (296.4, 175.9)
- added D16: WS2812C-2020, LED_SMD:LED_WS2812B-2020_PLCC4_2.0x2.0mm, F.Cu at (366.1, 198.9)
- added D17: WS2812C-2020, LED_SMD:LED_WS2812B-2020_PLCC4_2.0x2.0mm, F.Cu at (358.9, 191.2)
- added D18: WS2812C-2020, LED_SMD:LED_WS2812B-2020_PLCC4_2.0x2.0mm, F.Cu at (196.2, 179.7)
- added D19: WS2812C-2020, LED_SMD:LED_WS2812B-2020_PLCC4_2.0x2.0mm, F.Cu at (297.9, 162.1)
- added D2: WS2812C-2020, LED_SMD:LED_WS2812B-2020_PLCC4_2.0x2.0mm, F.Cu at (332.6, 186.4)
- added D20: WS2812C-2020, LED_SMD:LED_WS2812B-2020_PLCC4_2.0x2.0mm, F.Cu at (279.0, 169.5)
- added D21: WS2812C-2020, LED_SMD:LED_WS2812B-2020_PLCC4_2.0x2.0mm, F.Cu at (223.0, 208.5)
- added D22: WS2812C-2020, LED_SMD:LED_WS2812B-2020_PLCC4_2.0x2.0mm, F.Cu at (357.5, 220.0)
- added D23: WS2812C, LED_SMD:LED_WS2812B_PLCC4_5.0x5.0mm_P3.2mm, B.Cu at (225.5, 317.0)
- added D24: WS2812C, LED_SMD:LED_WS2812B_PLCC4_5.0x5.0mm_P3.2mm, B.Cu at (199.8, 291.0)
- added D25: WS2812C, LED_SMD:LED_WS2812B_PLCC4_5.0x5.0mm_P3.2mm, B.Cu at (174.0, 265.0)
- added D26: WS2812C, LED_SMD:LED_WS2812B_PLCC4_5.0x5.0mm_P3.2mm, B.Cu at (148.2, 239.0)
- added D27: WS2812C, LED_SMD:LED_WS2812B_PLCC4_5.0x5.0mm_P3.2mm, B.Cu at (122.5, 213.0)
- added D28: WS2812C, LED_SMD:LED_WS2812B_PLCC4_5.0x5.0mm_P3.2mm, B.Cu at (145.4, 188.7)
- added D29: WS2812C, LED_SMD:LED_WS2812B_PLCC4_5.0x5.0mm_P3.2mm, B.Cu at (171.8, 162.8)
- added D3: WS2812C-2020, LED_SMD:LED_WS2812B-2020_PLCC4_2.0x2.0mm, F.Cu at (361.0, 181.8)
- added D30: WS2812C, LED_SMD:LED_WS2812B_PLCC4_5.0x5.0mm_P3.2mm, B.Cu at (198.1, 137.0)
- added D31: WS2812C, LED_SMD:LED_WS2812B_PLCC4_5.0x5.0mm_P3.2mm, B.Cu at (224.4, 111.2)
- added D32: WS2812C, LED_SMD:LED_WS2812B_PLCC4_5.0x5.0mm_P3.2mm, B.Cu at (250.7, 85.3)
- added D33: WS2812C, LED_SMD:LED_WS2812B_PLCC4_5.0x5.0mm_P3.2mm, B.Cu at (277.0, 59.5)
- added D34: WS2812C, LED_SMD:LED_WS2812B_PLCC4_5.0x5.0mm_P3.2mm, B.Cu at (302.8, 85.1)
- added D35: WS2812C, LED_SMD:LED_WS2812B_PLCC4_5.0x5.0mm_P3.2mm, B.Cu at (328.6, 110.7)
- added D36: WS2812C, LED_SMD:LED_WS2812B_PLCC4_5.0x5.0mm_P3.2mm, B.Cu at (354.3, 136.2)
- added D37: WS2812C, LED_SMD:LED_WS2812B_PLCC4_5.0x5.0mm_P3.2mm, B.Cu at (380.1, 161.8)
- added D38: WS2812C, LED_SMD:LED_WS2812B_PLCC4_5.0x5.0mm_P3.2mm, B.Cu at (405.9, 187.4)
- added D39: WS2812C, LED_SMD:LED_WS2812B_PLCC4_5.0x5.0mm_P3.2mm, B.Cu at (431.6, 213.0)
- added D4: WS2812C-2020, LED_SMD:LED_WS2812B-2020_PLCC4_2.0x2.0mm, F.Cu at (243.7, 235.0)
- added D40: WS2812C, LED_SMD:LED_WS2812B_PLCC4_5.0x5.0mm_P3.2mm, B.Cu at (405.9, 239.0)
- added D41: WS2812C, LED_SMD:LED_WS2812B_PLCC4_5.0x5.0mm_P3.2mm, B.Cu at (380.1, 265.0)
- added D42: WS2812C, LED_SMD:LED_WS2812B_PLCC4_5.0x5.0mm_P3.2mm, B.Cu at (354.3, 291.0)
- added D43: WS2812C, LED_SMD:LED_WS2812B_PLCC4_5.0x5.0mm_P3.2mm, B.Cu at (328.6, 317.0)
- added D44: WS2812C-2020, LED_SMD:LED_WS2812B-2020_PLCC4_2.0x2.0mm, F.Cu at (220.4, 224.6)
- added D45: WS2812C-2020, LED_SMD:LED_WS2812B-2020_PLCC4_2.0x2.0mm, F.Cu at (351.1, 199.9)
- added D46: WS2812C-2020, LED_SMD:LED_WS2812B-2020_PLCC4_2.0x2.0mm, F.Cu at (362.5, 177.0)
- added D47: WS2812C-2020, LED_SMD:LED_WS2812B-2020_PLCC4_2.0x2.0mm, F.Cu at (277.0, 166.0)
- added D48: WS2812C-2020, LED_SMD:LED_WS2812B-2020_PLCC4_2.0x2.0mm, F.Cu at (219.0, 173.5)
- added D49: WS2812C-2020, LED_SMD:LED_WS2812B-2020_PLCC4_2.0x2.0mm, F.Cu at (356.0, 203.0)
- added D5: WS2812C-2020, LED_SMD:LED_WS2812B-2020_PLCC4_2.0x2.0mm, F.Cu at (205.5, 195.0)
- added D50: WS2812C-2020, LED_SMD:LED_WS2812B-2020_PLCC4_2.0x2.0mm, F.Cu at (352.1, 209.4)
- added D51: WS2812C-2020, LED_SMD:LED_WS2812B-2020_PLCC4_2.0x2.0mm, F.Cu at (310.6, 190.9)
- added D52: WS2812C-2020, LED_SMD:LED_WS2812B-2020_PLCC4_2.0x2.0mm, F.Cu at (209.5, 185.0)
- added D53: WS2812C-2020, LED_SMD:LED_WS2812B-2020_PLCC4_2.0x2.0mm, F.Cu at (225.5, 172.5)
- added D54: WS2812C-2020, LED_SMD:LED_WS2812B-2020_PLCC4_2.0x2.0mm, F.Cu at (306.0, 219.5)
- added D55: WS2812C-2020, LED_SMD:LED_WS2812B-2020_PLCC4_2.0x2.0mm, F.Cu at (220.0, 188.5)
- added D56: WS2812C-2020, LED_SMD:LED_WS2812B-2020_PLCC4_2.0x2.0mm, F.Cu at (227.9, 244.4)
- added D57: WS2812C-2020, LED_SMD:LED_WS2812B-2020_PLCC4_2.0x2.0mm, F.Cu at (301.5, 197.5)
- added D58: WS2812C-2020, LED_SMD:LED_WS2812B-2020_PLCC4_2.0x2.0mm, F.Cu at (290.1, 243.9)
- added D59: WS2812C-2020, LED_SMD:LED_WS2812B-2020_PLCC4_2.0x2.0mm, F.Cu at (296.5, 238.0)
- added D6: WS2812C-2020, LED_SMD:LED_WS2812B-2020_PLCC4_2.0x2.0mm, F.Cu at (297.5, 186.0)
- added D60: WS2812C-2020, LED_SMD:LED_WS2812B-2020_PLCC4_2.0x2.0mm, F.Cu at (274.5, 176.0)
- added D61: WS2812C-2020, LED_SMD:LED_WS2812B-2020_PLCC4_2.0x2.0mm, F.Cu at (378.5, 249.5)
- added D62: WS2812C-2020, LED_SMD:LED_WS2812B-2020_PLCC4_2.0x2.0mm, F.Cu at (201.5, 164.5)
- added D63: WS2812C-2020, LED_SMD:LED_WS2812B-2020_PLCC4_2.0x2.0mm, F.Cu at (304.0, 214.5)
- added D64: WS2812C-2020, LED_SMD:LED_WS2812B-2020_PLCC4_2.0x2.0mm, F.Cu at (279.5, 180.0)
- added D7: WS2812C-2020, LED_SMD:LED_WS2812B-2020_PLCC4_2.0x2.0mm, F.Cu at (330.2, 195.8)
- added D8: WS2812C-2020, LED_SMD:LED_WS2812B-2020_PLCC4_2.0x2.0mm, F.Cu at (353.5, 174.0)
- added D9: WS2812C-2020, LED_SMD:LED_WS2812B-2020_PLCC4_2.0x2.0mm, F.Cu at (341.0, 190.0)
- added J1: OLED Display, Connector_PinHeader_2.54mm:PinHeader_1x04_P2.54mm_Vertical, F.Cu at (151.8, 196.7)
- added J2: U1_Header_1, Connector_PinSocket_2.54mm:PinSocket_1x07_P2.54mm_Vertical, F.Cu at (314.1, 332.4)
- added J3: U1_Header_2, Connector_PinSocket_2.54mm:PinSocket_1x07_P2.54mm_Vertical, F.Cu at (294.1, 352.4)
- added R1: 10k, Resistor_THT:R_Axial_DIN0207_L6.3mm_D2.5mm_P7.62mm_Horizontal, F.Cu at (145.2, 211.5)
- added R2: 10k, Resistor_THT:R_Axial_DIN0207_L6.3mm_D2.5mm_P7.62mm_Horizontal, F.Cu at (163.2, 211.5)
- added R3: 10k, Resistor_THT:R_Axial_DIN0207_L6.3mm_D2.5mm_P7.62mm_Horizontal, F.Cu at (180.7, 211.5)
- added SW1: SW_SPDT, Button_Switch_THT:SW_Slide_SPDT_Angled_CK_OS102011MA1Q, F.Cu at (321.2, 329.0)
- added SW2: SW_Push, Button_Switch_THT:SW_PUSH-12mm, F.Cu at (142.8, 220.5)
- added SW3: SW_Push, Button_Switch_THT:SW_PUSH-12mm, F.Cu at (160.8, 220.5)
- added SW4: SW_Push, Button_Switch_THT:SW_PUSH-12mm, F.Cu at (178.8, 220.5)
- moved U1 23.9 mm to (298.5, 337.0), turned to -135 degrees
- moved G*** 7.37 mm to (287.0, 198.0)
Connections:
- U1 pad 1: unconnected-(U1-PA02_A0_D0-Pad1) -> BAT_SW
- U1 pad 10: unconnected-(U1-PA5_A9_D9_MISO-Pad10) -> BTN_CENTER
- U1 pad 11: unconnected-(U1-PA6_A10_D10_MOSI-Pad11) -> BTN_LEFT
- U1 pad 12: unconnected-(U1-3V3-Pad12) -> +3V3
- U1 pad 13: unconnected-(U1-GND-Pad13) -> GND
- U1 pad 14: unconnected-(U1-5V-Pad14) -> +5V
- U1 pad 2: unconnected-(U1-PA4_A1_D1-Pad2) -> CITY_LEDS
- U1 pad 3: unconnected-(U1-PA10_A2_D2-Pad3) -> BOTTOM_LEDS
- U1 pad 4: unconnected-(U1-PA11_A3_D3-Pad4) -> A3_D3
- U1 pad 5: unconnected-(U1-PA8_A4_D4_SDA-Pad5) -> DISP_SDA
- U1 pad 6: unconnected-(U1-PA9_A5_D5_SCL-Pad6) -> DISP_SCL
- U1 pad 7: unconnected-(U1-PB08_A6_TX-Pad7) -> A6_TX
- U1 pad 8: unconnected-(U1-PB09_D7_RX-Pad8) -> D7_RX
- U1 pad 9: unconnected-(U1-PA7_A8_D8_SCK-Pad9) -> BTN_RIGHT
Other:
- copper layers 2 -> 4
- board text added: "ANTENNA"
- board text added: "Algiers"
- board text added: "Bangkok"
- board text added: "Beijing"
- board text added: "Bogotá"
- board text added: "Buenos Aires"
- board text added: "Cairo"
- board text added: "Cape Town"
- board text added: "Chicago"
- board text added: "Chongqing"
- board text added: "Dar es Salaam"
- board text added: "Delhi"
- board text added: "Dhaka"
- board text added: "Ho Chi Minh City"
- board text added: "Hong Kong"
- board text added: "Houston"
- board text added: "Istanbul"
- board text added: "Jakarta"
- board text added: "Johannesburg"
- board text added: "Karachi"
- board text added: "Khartoum"
- board text added: "Kuala Lumpur"
- board text added: "Lima"
- board text added: "London"
- board text added: "Los Angeles"
- board text added: "Madrid"
- board text added: "Manila"
- board text added: "Mexico City"
- board text added: "Miami"
- board text added: "Moscow"
- board text added: "Mumbai"
- board text added: "Nairobi"
- board text added: "New York"
- board text added: "Paris"
- board text added: "Riyadh"
- board text added: "Santiago"
- board text added: "Seoul"
- board text added: "Shanghai"
- board text added: "Sydney"
- board text added: "São Paulo"
- board text added: "Tehran"
- board text added: "Tokyo"
- board text added: "Toronto"
- board text added: "Vancouver"
- board text added: "https://github.com/peter-lamantia/gradcap-threatmap"

Commit message: Almost there
Parts:
- removed D1: WS2812C-2020, LED_SMD:LED_WS2812B-2020_PLCC4_2.0x2.0mm
- removed the D61 at (378.5, 249.5)
- added D64: WS2812C-2020, LED_SMD:LED_WS2812B-2020_PLCC4_2.0x2.0mm, F.Cu at (369.9, 176.6)
- added D65: WS2812C-2020, LED_SMD:LED_WS2812B-2020_PLCC4_2.0x2.0mm, F.Cu at (378.5, 248.4)
- turned D10 to 180 degrees
- turned D12 to 180 degrees
- turned D13 to 180 degrees
- turned D14 to 180 degrees
- turned D19 to 180 degrees
- turned D2 to 180 degrees
- turned D20 to 180 degrees
- turned D21 to 180 degrees
- turned D44 to 180 degrees
- turned D46 to 180 degrees
- turned D5 to 180 degrees
- turned D50 to 180 degrees
- turned D51 to 180 degrees
- turned D52 to 180 degrees
- turned D53 to 180 degrees
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- renumbered D21 to D10, D44 to D11, D56 to D12, D4 to D14, D20 to D15, D64 to D16, D47 to D17, D60 to D18, D58 to D19, D62 to D2, D19 to D20, D11 to D21, D6 to D22, D52 to D3, D18 to D4, D15 to D44, D57 to D45, D51 to D46, D63 to D47, D59 to D48, D54 to D49, D9 to D50, D12 to D51, D2 to D52, D7 to D53, D46 to D54, D14 to D55, D8 to D56, D3 to D57, D45 to D58, D49 to D59, D48 to D6, D50 to D60, D16 to D61, D17 to D62, D22 to D63, D10 to D7, D55 to D8, D53 to D9
Connections:
- D10 pad 1: Net-(D21-DOUT) -> Net-(D10-DOUT)
- D10 pad 3: Net-(D20-DOUT) -> Net-(D10-DIN)
- D10 pad 4: Net-(D21-VDD) -> BAT_SW
- D11 pad 1: Net-(D44-DOUT) -> Net-(D11-DOUT)
- D11 pad 3: Net-(D22-DOUT) -> Net-(D10-DOUT)
- D11 pad 4: Net-(D21-VDD) -> BAT_SW
- D12 pad 1: Net-(D56-DOUT) -> Net-(D12-DOUT)
- D12 pad 3: Net-(D55-DOUT) -> Net-(D11-DOUT)
- D12 pad 4: Net-(D21-VDD) -> BAT_SW
- D14 pad 1: Net-(D4-DOUT) -> Net-(D14-DOUT)
- D14 pad 3: Net-(D3-DOUT) -> Net-(D13-DOUT)
- D15 pad 1: Net-(D20-DOUT) -> Net-(D15-DOUT)
- D15 pad 3: Net-(D19-DOUT) (its old number) -> Net-(D15-DIN)
- D16 pad 1: unconnected-(D64-DOUT-Pad1) -> Net-(D16-DOUT)
- D16 pad 2: GND -> BAT_SW
- D16 pad 3: Net-(D63-DOUT) -> Net-(D16-DIN)
- D16 pad 4: Net-(D21-VDD) -> GND
- D17 pad 1: Net-(D47-DOUT) -> Net-(D17-DOUT)
- D17 pad 3: Net-(D46-DOUT) -> Net-(D15-DOUT)
- D17 pad 4: Net-(D21-VDD) -> BAT_SW
- D18 pad 1: Net-(D60-DOUT) -> Net-(D15-DIN)
- D18 pad 3: Net-(D59-DOUT) -> Net-(D16-DOUT)
- D18 pad 4: Net-(D21-VDD) -> BAT_SW
- D19 pad 3: Net-(D57-DOUT) -> Net-(D14-DOUT)
- D19 pad 4: Net-(D21-VDD) -> BAT_SW
- D2 pad 1: Net-(D62-DOUT) -> Net-(D2-DOUT)
- D2 pad 3: Net-(D61-DOUT) -> CITY_LEDS
- D2 pad 4: Net-(D21-VDD) -> BAT_SW
- D20 pad 1: Net-(D19-DOUT) (its old number) -> Net-(D20-DOUT)
- D20 pad 3: Net-(D18-DOUT) -> Net-(D17-DOUT)
- D21 pad 1: Net-(D11-DOUT) -> Net-(D21-DOUT)
- D21 pad 3: Net-(D10-DOUT) -> Net-(D21-DIN)
- D22 pad 1: Net-(D6-DOUT) -> Net-(D16-DIN)
- D22 pad 3: Net-(D5-DOUT) -> Net-(D22-DIN)
- D3 pad 1: Net-(D52-DOUT) -> Net-(D3-DOUT)
- D3 pad 3: Net-(D51-DOUT) -> Net-(D3-DIN)
- D3 pad 4: Net-(D21-VDD) -> BAT_SW
- D4 pad 1: Net-(D18-DOUT) -> Net-(D4-DOUT)
- D4 pad 3: Net-(D17-DOUT) -> Net-(D3-DOUT)
- D44 pad 1: Net-(D15-DOUT) -> Net-(D21-DIN)
- D44 pad 3: Net-(D14-DOUT) -> Net-(D20-DOUT)
- D45 pad 1: Net-(D57-DOUT) -> Net-(D22-DIN)
- D45 pad 3: Net-(D56-DOUT) -> Net-(D45-DIN)
- D45 pad 4: Net-(D21-VDD) -> BAT_SW
- D46 pad 1: Net-(D51-DOUT) -> Net-(D46-DOUT)
- D46 pad 3: Net-(D50-DOUT) -> Net-(D21-DOUT)
- D46 pad 4: Net-(D21-VDD) -> BAT_SW
- D47 pad 1: Net-(D63-DOUT) -> Net-(D45-DIN)
- D47 pad 3: Net-(D62-DOUT) -> Net-(D47-DIN)
- D47 pad 4: Net-(D21-VDD) -> BAT_SW
- D48 pad 1: Net-(D59-DOUT) -> Net-(D48-DOUT)
- D48 pad 4: Net-(D21-VDD) -> BAT_SW
- D49 pad 1: Net-(D54-DOUT) -> Net-(D47-DIN)
- D49 pad 3: Net-(D53-DOUT) -> Net-(D48-DOUT)
- D49 pad 4: Net-(D21-VDD) -> BAT_SW
- D5 pad 1: Net-(D5-DOUT) -> Net-(D10-DIN)
- D50 pad 1: Net-(D10-DIN) -> Net-(D50-DOUT)
- D50 pad 3: Net-(D8-DOUT) -> Net-(D50-DIN)
- D51 pad 1: Net-(D12-DOUT) -> Net-(D51-DOUT)
- D51 pad 3: Net-(D11-DOUT) -> Net-(D46-DOUT)
- D52 pad 1: Net-(D2-DOUT) -> Net-(D52-DOUT)
- D52 pad 3: Net-(D1-DOUT) -> Net-(D51-DOUT)
- D53 pad 1: Net-(D7-DOUT) -> Net-(D50-DIN)
- D53 pad 3: Net-(D6-DOUT) -> Net-(D52-DOUT)
- D54 pad 1: Net-(D46-DOUT) -> Net-(D54-DOUT)
- D54 pad 3: Net-(D45-DOUT) -> Net-(D54-DIN)
- D54 pad 4: Net-(D21-VDD) -> BAT_SW
- D55 pad 1: Net-(D14-DOUT) -> Net-(D55-DOUT)
- D55 pad 3: Net-(D13-DOUT) -> Net-(D50-DOUT)
- D56 pad 1: Net-(D8-DOUT) -> Net-(D54-DIN)
- D56 pad 3: Net-(D7-DOUT) -> Net-(D55-DOUT)
- D57 pad 1: Net-(D3-DOUT) -> Net-(D57-DOUT)
- D57 pad 3: Net-(D2-DOUT) -> Net-(D57-DIN)
- D58 pad 1: Net-(D45-DOUT) -> Net-(D58-DOUT)
- D58 pad 3: Net-(D44-DOUT) -> Net-(D58-DIN)
- D58 pad 4: Net-(D21-VDD) -> BAT_SW
- D59 pad 1: Net-(D49-DOUT) -> Net-(D58-DIN)
- D59 pad 3: Net-(D48-DOUT) -> Net-(D59-DIN)
- D59 pad 4: Net-(D21-VDD) -> BAT_SW
- D6 pad 1: Net-(D48-DOUT) -> Net-(D6-DOUT)
- D6 pad 3: Net-(D47-DOUT) -> Net-(D2-DOUT)
- D6 pad 4: Net-(D21-VDD) -> BAT_SW
- D60 pad 1: Net-(D50-DOUT) -> Net-(D60-DOUT)
- D60 pad 3: Net-(D49-DOUT) -> Net-(D58-DOUT)
- D60 pad 4: Net-(D21-VDD) -> BAT_SW
- D61 pad 1: Net-(D16-DOUT) -> Net-(D59-DIN)
- D61 pad 3: Net-(D15-DOUT) -> Net-(D61-DIN)
- D62 pad 1: Net-(D17-DOUT) -> Net-(D61-DIN)
- D62 pad 3: Net-(D16-DOUT) -> Net-(D57-DOUT)
- D63 pad 1: Net-(D22-DOUT) -> Net-(D63-DOUT)
- D63 pad 3: Net-(D21-DOUT) -> Net-(D60-DOUT)
- D63 pad 4: Net-(D21-VDD) -> BAT_SW
- D7 pad 1: Net-(D10-DOUT) -> Net-(D7-DOUT)
- D7 pad 3: Net-(D10-DIN) -> Net-(D7-DIN)
- D8 pad 1: Net-(D55-DOUT) -> Net-(D3-DIN)
- D8 pad 3: Net-(D54-DOUT) -> Net-(D7-DOUT)
- D8 pad 4: Net-(D21-VDD) -> BAT_SW
- D9 pad 1: Net-(D53-DOUT) -> Net-(D7-DIN)
- D9 pad 3: Net-(D52-DOUT) -> Net-(D6-DOUT)
- D9 pad 4: Net-(D21-VDD) -> BAT_SW
- SW2 pad 2: +BATT -> BAT_SW
- SW3 pad 2: +BATT -> BAT_SW
- SW4 pad 2: +BATT -> BAT_SW
Routing:
- net GND: track 0.00 -> 1646.7 mm, vias 0 -> 5
- net BAT_SW: track 0.00 -> 1630.3 mm, vias 0 -> 8
- net CITY_LEDS: track 0.00 -> 245.2 mm
- net BTN_LEFT: track 0.00 -> 231.5 mm, vias 0 -> 2
- net BTN_CENTER: track 0.00 -> 229.0 mm, vias 0 -> 2
- net DISP_SDA: track 0.00 -> 224.2 mm
- net DISP_SCL: track 0.00 -> 223.0 mm
- net BTN_RIGHT: track 0.00 -> 187.0 mm
- net BOTTOM_LEDS: track 0.00 -> 91.1 mm
- net Net-(D14-DOUT): track 0.00 -> 47.8 mm
- net Net-(D32-DOUT): track 0.00 -> 35.6 mm
- net Net-(D26-DOUT): track 0.00 -> 35.4 mm
- net Net-(D63-DOUT): track 0.00 -> 35.3 mm
- net Net-(D38-DOUT): track 0.00 -> 35.2 mm
- net Net-(D30-DOUT): track 0.00 -> 33.2 mm
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Other:
- copper layers 4 -> 2
- board text added: "Peter LaMantia | M.S. Cybersecurity - 2025 -"
- board text added: "https://github.com/peter-lamantia/ gradcap-threatmap"
- board text removed: "Vancouver"
- board text removed: "https://github.com/peter-lamantia/gradcap-threatmap"

Commit message: Updated pcb
Parts:
- added BAT+: TestPoint, TestPoint:TestPoint_Keystone_5015_Micro_Mini, B.Cu at (365.8, 274.8)
- added GND: TestPoint, TestPoint:TestPoint_Keystone_5015_Micro_Mini, B.Cu at (360.5, 274.8)
- moved D27 120.1 mm to (169.3, 323.6), turned to -45 degrees
- moved D33 116.6 mm to (170.0, 105.8), turned to -135 degrees
- moved D39 116.5 mm to (387.9, 105.0), turned to 135 degrees
- moved J3 108.2 mm to (389.2, 300.9), turned to -90 degrees
- moved SW2 104.8 mm to (188.9, 314.6), turned to 45 degrees
- moved D28 104.0 mm to (168.3, 290.2), turned to -90 degrees
- moved R1 102.7 mm to (184.3, 306.5), turned to 45 degrees
- moved D26 102.5 mm to (205.9, 323.8), turned to 0 degrees
- moved D32 99.3 mm to (169.6, 142.7), turned to -90 degrees
- moved D40 99.0 mm to (388.0, 141.6), turned to 90 degrees
- moved D34 98.6 mm to (206.3, 105.7), turned to 180 degrees
- moved D38 98.6 mm to (351.6, 105.1), turned to 180 degrees
- moved J1 98.4 mm to (178.4, 291.4), turned to 45 degrees
- moved U1 96.9 mm to (381.4, 286.8), turned to -90 degrees
- moved J2 96.0 mm to (389.2, 272.6), turned to -90 degrees
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Connections:
- net +3V3 renamed U1_3V3
- net +5V renamed U1_5V
Routing:
- net BAT_SW: track 1630.3 -> 1660.4 mm
- net GND: track 1646.7 -> 1673.2 mm, vias 5 -> 30
- added copper zone on B.Cu, net GND
- added copper zone on F.Cu, net GND
Other:
- board size 332.3 x 332.3 mm -> 235 x 235 mm
- board text added: "Vancouver"
