File: pcb/pcb.kicad_sch (KiCad schematic)
At the start: 3 parts, among them J1 Conn_01x02_MountingPin, U1 MOUDLE-SEEEDUINO-XIAO-ESP32S3

Commit message: Moving along
Parts:
- removed J1: Conn_01x02_MountingPin, symbol Connector_Generic_MountingPin:Conn_01x02_MountingPin
- added BT1: Battery Connector, Connector_JST:JST_PH_S2B-PH-K_1x02_P2.00mm_Horizontal, symbol Device:Battery_Cell
- added D10, D11, D12, D13, D14, D15, D16, D17, D18, D19, D2, D20, D21, D22, D3, D4, D44, D45, D46, D47, D48, D49, D5, D50, D51, D52, D53, D54, D55, D56, D57, D58, D59, D6, D60, D61, D62, D63, D64, D7, D8, D9: WS2812C-2020, LED_SMD:LED_WS2812B-2020_PLCC4_2.0x2.0mm, symbol LED:WS2812B-2020
- added D23, D24, D25, D26, D27, D28, D29, D30, D31, D32, D33, D34, D35, D36, D37, D38, D39, D40, D41, D42, D43: WS2812C, LED_SMD:LED_WS2812B_PLCC4_5.0x5.0mm_P3.2mm, symbol LED:WS2812B
- added J1: OLED Display, Connector_PinHeader_2.54mm:PinHeader_1x04_P2.54mm_Vertical, symbol Connector:Conn_01x04_Pin
- added J2: U1_Header_1, Connector_PinSocket_2.54mm:PinSocket_1x07_P2.54mm_Vertical, symbol Connector:Conn_01x07_Pin
- added J3: U1_Header_2, Connector_PinSocket_2.54mm:PinSocket_1x07_P2.54mm_Vertical, symbol Connector:Conn_01x07_Pin
- added R1, R2, R3: 10k, Resistor_THT:R_Axial_DIN0207_L6.3mm_D2.5mm_P7.62mm_Horizontal, symbol Device:R_Small
- added SW1: SW_SPDT, Button_Switch_THT:SW_Slide_SPDT_Angled_CK_OS102011MA1Q, symbol Switch:SW_SPDT
- added SW2, SW3, SW4: SW_Push, Button_Switch_THT:SW_PUSH-12mm, symbol Switch:SW_Push
- D1: value WS2812B-2020 -> WS2812C-2020
Connections:
- net BAT_SW: now reaches U1.1 (PA02_A0_D0)
- net BAT_SW: now also D1.4 (VDD), D10.4 (VDD), D11.4 (VDD), D12.4 (VDD), D13.4 (VDD), D14.4 (VDD), D15.4 (VDD), D16.4 (VDD), D17.4 (VDD), D18.4 (VDD), D19.4 (VDD), D2.4 (VDD), D20.4 (VDD), D23.1 (VDD), D24.1 (VDD), D25.1 (VDD), D26.1 (VDD), D27.1 (VDD), D28.1 (VDD), D29.1 (VDD), D3.4 (VDD), D30.1 (VDD), D31.1 (VDD), D32.1 (VDD), D33.1 (VDD), D34.1 (VDD), D35.1 (VDD), D36.1 (VDD), D37.1 (VDD), D38.1 (VDD), D39.1 (VDD), D4.4 (VDD), D40.1 (VDD), D41.1 (VDD), D42.1 (VDD), D43.1 (VDD), D5.4 (VDD), D6.4 (VDD), D7.4 (VDD), D8.4 (VDD), D9.4 (VDD), J1.2 (Pin_2), J2.1 (Pin_1), SW1.1 (A)
- net BTN_CENTER: now reaches U1.10 (PA5_A9_D9_MISO)
- net BTN_CENTER: now also J3.5 (Pin_5), R2.1, SW3.1
- net BTN_LEFT: now reaches U1.11 (PA6_A10_D10_MOSI)
- net BTN_LEFT: now also J3.4 (Pin_4), R1.1, SW2.1
- net +3V3: now reaches U1.12 (3V3)
- net +3V3: now also J3.3 (Pin_3)
- net GND: now reaches U1.13 (GND)
- net GND: now also D1.2 (VSS), BT1.2 (-), D10.2 (VSS), D11.2 (VSS), D12.2 (VSS), D13.2 (VSS), D14.2 (VSS), D15.2 (VSS), D16.2 (VSS), D17.2 (VSS), D18.2 (VSS), D19.2 (VSS), D2.2 (VSS), D20.2 (VSS), D21.2 (VSS), D22.2 (VSS), D23.3 (VSS), D24.3 (VSS), D25.3 (VSS), D26.3 (VSS), D27.3 (VSS), D28.3 (VSS), D29.3 (VSS), D3.2 (VSS), D30.3 (VSS), D31.3 (VSS), D32.3 (VSS), D33.3 (VSS), D34.3 (VSS), D35.3 (VSS), D36.3 (VSS), D37.3 (VSS), D38.3 (VSS), D39.3 (VSS), D4.2 (VSS), D40.3 (VSS), D41.3 (VSS), D42.3 (VSS), D43.3 (VSS), D44.2 (VSS), D45.2 (VSS), D46.2 (VSS), D47.2 (VSS), D48.2 (VSS), D49.2 (VSS), D5.2 (VSS), D50.2 (VSS), D51.2 (VSS), D52.2 (VSS), D53.2 (VSS), D54.2 (VSS), D55.2 (VSS), D56.2 (VSS), D57.2 (VSS), D58.2 (VSS), D59.2 (VSS), D6.2 (VSS), D60.2 (VSS), D61.2 (VSS), D62.2 (VSS), D63.2 (VSS), D64.2 (VSS), D7.2 (VSS), D8.2 (VSS), D9.2 (VSS), J1.1 (Pin_1), J3.2 (Pin_2), R1.2, R2.2, R3.2
- net +5V: now reaches U1.14 (5V)
- net +5V: now also J3.1 (Pin_1)
- net CITY_LEDS: now reaches U1.2 (PA4_A1_D1)
- net CITY_LEDS: now also D1.3 (DIN), J2.2 (Pin_2)
- net BOTTOM_LEDS: now reaches U1.3 (PA10_A2_D2)
- net BOTTOM_LEDS: now also D23.4 (DIN), J2.3 (Pin_3)
- net A3_D3: now reaches U1.4 (PA11_A3_D3)
- net A3_D3: now also J2.4 (Pin_4)
- net DISP_SDA: now reaches U1.5 (PA8_A4_D4_SDA)
- net DISP_SDA: now also J1.4 (Pin_4), J2.5 (Pin_5)
- net DISP_SCL: now reaches U1.6 (PA9_A5_D5_SCL)
- net DISP_SCL: now also J1.3 (Pin_3), J2.6 (Pin_6)
- net A6_TX: now reaches U1.7 (PB08_A6_TX)
- net A6_TX: now also J2.7 (Pin_7)
- net D7_RX: now reaches U1.8 (PB09_D7_RX)
- net D7_RX: now also J3.7 (Pin_7)
- net BTN_RIGHT: now reaches U1.9 (PA7_A8_D8_SCK)
- net BTN_RIGHT: now also J3.6 (Pin_6), R3.1, SW4.1
- net at D1.1 (DOUT): now also D2.3 (DIN)
- new net: D28.2 (DOUT), D29.4 (DIN)
- new net: D27.2 (DOUT), D28.4 (DIN)
- new net: D42.2 (DOUT), D43.4 (DIN)
- new net: D53.1 (DOUT), D54.3 (DIN)
- new net: D52.1 (DOUT), D53.3 (DIN)
- new net: D21.4 (VDD), D22.4 (VDD), D44.4 (VDD), D45.4 (VDD), D46.4 (VDD), D47.4 (VDD), D48.4 (VDD), D49.4 (VDD), D50.4 (VDD), D51.4 (VDD), D52.4 (VDD), D53.4 (VDD), D54.4 (VDD), D55.4 (VDD), D56.4 (VDD), D57.4 (VDD), D58.4 (VDD), D59.4 (VDD), D60.4 (VDD), D61.4 (VDD), D62.4 (VDD), D63.4 (VDD), D64.4 (VDD)
- new net: D32.2 (DOUT), D33.4 (DIN)
- new net: D31.2 (DOUT), D32.4 (DIN)
- new net: D20.1 (DOUT), D21.3 (DIN)
- new net: D19.1 (DOUT), D20.3 (DIN)
- new net: D25.2 (DOUT), D26.4 (DIN)
- new net: D24.2 (DOUT), D25.4 (DIN)
- new net: D10.1 (DOUT), D11.3 (DIN)
- new net: D10.3 (DIN), D9.1 (DOUT)
- new net: D29.2 (DOUT), D30.4 (DIN)
- new net: D8.1 (DOUT), D9.3 (DIN)
- new net: D23.2 (DOUT), D24.4 (DIN)
- new net: D7.1 (DOUT), D8.3 (DIN)
- new net: D49.1 (DOUT), D50.3 (DIN)
- new net: D48.1 (DOUT), D49.3 (DIN)
- new net: D36.2 (DOUT), D37.4 (DIN)
- new net: D35.2 (DOUT), D36.4 (DIN)
- new net: D26.2 (DOUT), D27.4 (DIN)
- new net: D22.1 (DOUT), D44.3 (DIN)
- new net: D21.1 (DOUT), D22.3 (DIN)
- new net: D12.1 (DOUT), D13.3 (DIN)
- new net: D11.1 (DOUT), D12.3 (DIN)
- new net: D57.1 (DOUT), D58.3 (DIN)
- new net: D56.1 (DOUT), D57.3 (DIN)
- new net: D18.1 (DOUT), D19.3 (DIN)
- new net: D33.2 (DOUT), D34.4 (DIN)
- new net: D17.1 (DOUT), D18.3 (DIN)
- new net: D16.1 (DOUT), D17.3 (DIN)
- new net: D59.1 (DOUT), D60.3 (DIN)
- new net: D58.1 (DOUT), D59.3 (DIN)
- new net: D15.1 (DOUT), D16.3 (DIN)
- new net: D45.1 (DOUT), D46.3 (DIN)
- new net: D44.1 (DOUT), D45.3 (DIN)
- new net: D4.1 (DOUT), D5.3 (DIN)
- new net: D3.1 (DOUT), D4.3 (DIN)
- new net: D6.1 (DOUT), D7.3 (DIN)
- new net: D5.1 (DOUT), D6.3 (DIN)
- new net: D61.1 (DOUT), D62.3 (DIN)
- new net: D60.1 (DOUT), D61.3 (DIN)
- new net: D46.1 (DOUT), D47.3 (DIN)
- new net: D62.1 (DOUT), D63.3 (DIN)
- new net: D50.1 (DOUT), D51.3 (DIN)
- new net: D39.2 (DOUT), D40.4 (DIN)
- new net: D38.2 (DOUT), D39.4 (DIN)
- new net: D51.1 (DOUT), D52.3 (DIN)
- new net: D13.1 (DOUT), D14.3 (DIN)
- new net: D54.1 (DOUT), D55.3 (DIN)
- new net: D41.2 (DOUT), D42.4 (DIN)
- new net: D34.2 (DOUT), D35.4 (DIN)
- new net: D63.1 (DOUT), D64.3 (DIN)
- new net: D2.1 (DOUT), D3.3 (DIN)
- new net: D37.2 (DOUT), D38.4 (DIN)
- new net: D47.1 (DOUT), D48.3 (DIN)
- new net: D30.2 (DOUT), D31.4 (DIN)
- new net: D40.2 (DOUT), D41.4 (DIN)
- new net: D14.1 (DOUT), D15.3 (DIN)
- new net: D55.1 (DOUT), D56.3 (DIN)
- new net +BATT: BT1.1 (+), SW1.2 (B), SW2.2, SW3.2, SW4.2
- no-connect marks 0 -> 3
Other:
- note added: "The 10k resistor pulls the value low when the switch is off."
- note added: "WS2812C-2020 LEDs use 1/3 of the power of WS2812B. They are the same package and protocol."
- moved on the sheet: D1, U1

Commit message: Almost there
Parts:
- renumbered D1 to D65
Connections:
- net +BATT: no longer SW2.2, SW3.2, SW4.2
- net BAT_SW: now also D16.2 (VSS), D21.4 (VDD), D22.4 (VDD), D44.4 (VDD), D45.4 (VDD), D46.4 (VDD), D47.4 (VDD), D48.4 (VDD), D49.4 (VDD), D50.4 (VDD), D51.4 (VDD), D52.4 (VDD), D53.4 (VDD), D54.4 (VDD), D55.4 (VDD), D56.4 (VDD), D57.4 (VDD), D58.4 (VDD), D59.4 (VDD), D60.4 (VDD), D61.4 (VDD), D62.4 (VDD), D63.4 (VDD), D64.4 (VDD), SW2.2, SW3.2, SW4.2; no longer D16.4 (VDD)
- net CITY_LEDS: now also D2.3 (DIN); no longer D65.3 (DIN)
- net GND: now also D16.4 (VDD); no longer D16.2 (VSS)
- net at D53.1 (DOUT): now also D50.3 (DIN); no longer D54.3 (DIN)
- net at D20.1 (DOUT): now also D44.3 (DIN); no longer D21.3 (DIN)
- net at D20.3 (DIN): now also D17.1 (DOUT); no longer D19.1 (DOUT)
- net at D10.3 (DIN): now also D5.1 (DOUT); no longer D9.1 (DOUT)
- net at D9.3 (DIN): now also D6.1 (DOUT); no longer D8.1 (DOUT)
- net at D49.1 (DOUT): now also D47.3 (DIN); no longer D50.3 (DIN)
- net at D22.1 (DOUT): now also D16.3 (DIN); no longer D44.3 (DIN)
- net at D22.3 (DIN): now also D45.1 (DOUT); no longer D21.1 (DOUT)
- net at D57.1 (DOUT): now also D62.3 (DIN); no longer D58.3 (DIN)
- net at D57.3 (DIN): now also D64.1 (DOUT); no longer D56.1 (DOUT)
- net at D19.3 (DIN): now also D14.1 (DOUT); no longer D18.1 (DOUT)
- net at D18.3 (DIN): now also D16.1 (DOUT); no longer D17.1 (DOUT)
- net at D17.3 (DIN): now also D15.1 (DOUT); no longer D16.1 (DOUT)
- net at D59.1 (DOUT): now also D58.3 (DIN); no longer D60.3 (DIN)
- net at D59.3 (DIN): now also D61.1 (DOUT); no longer D58.1 (DOUT)
- net at D46.3 (DIN): now also D21.1 (DOUT); no longer D45.1 (DOUT)
- net at D45.3 (DIN): now also D47.1 (DOUT); no longer D44.1 (DOUT)
- net at D7.3 (DIN): now also D9.1 (DOUT); no longer D6.1 (DOUT)
- net at D6.3 (DIN): now also D2.1 (DOUT); no longer D5.1 (DOUT)
- net at D61.3 (DIN): now also D62.1 (DOUT); no longer D60.1 (DOUT)
- net at D46.1 (DOUT): now also D51.3 (DIN); no longer D47.3 (DIN)
- net at D63.3 (DIN): now also D60.1 (DOUT); no longer D62.1 (DOUT)
- net at D50.1 (DOUT): now also D55.3 (DIN); no longer D51.3 (DIN)
- net at D54.1 (DOUT): now also D64.3 (DIN); no longer D55.3 (DIN)
- net at D63.1 (DOUT): now also D65.3 (DIN); no longer D64.3 (DIN)
- net at D3.3 (DIN): now also D8.1 (DOUT); no longer D2.1 (DOUT)
- net at D65.1 (DOUT): no longer D2.3 (DIN)
- net at D48.3 (DIN): now also D19.1 (DOUT); no longer D47.1 (DOUT)
- net at D15.3 (DIN): now also D18.1 (DOUT); no longer D14.1 (DOUT)
- new net: D54.3 (DIN), D56.1 (DOUT)
- new net: D58.1 (DOUT), D60.3 (DIN)
- new net: D21.3 (DIN), D44.1 (DOUT)
Other:
- moved on the sheet: BT1, D10, D11, D12, D13, D14, D15, D16, D17, D18, D19, D2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

Commit message: Updated pcb
Parts:
- added TP2, TP3: TestPoint, TestPoint:TestPoint_Keystone_5015_Micro_Mini, symbol Connector:TestPoint
Connections:
- net BAT_SW: now also TP2.1
- net GND: now also TP3.1
- net +3V3 renamed U1_3V3
- net +5V renamed U1_5V
Other:
- moved on the sheet: BT1, SW1
